File: Amiga500.kicad_pcb (KiCad board)
At the start: 2 copper layers, 365.8 x 254 mm, 370 parts, among them CN1 LEFT_JOY, CN10 COMPOSITE, CN11 INTERNAL_FLOPPY, CN12 FLOPPY_POWER, CN13 KEYBOARD, CN14 IDE_POWER, CN15 IDE_I/F, CN2 RIGHT_JOY, CN3 RIGHT, CN4 LEFT, CN5 EXTFLOPPY_DB23F, CN6 SERIAL_DB25M, CN7 PARALLEL_DB25F, CN8 POWER, CN9 VIDEO_DB23M, J90 DRIVE_SWITCHER, J91 Dispatcher_3to1, J92 Dispatcher_3to1, J93 Dispatcher_3to1, J99 CONN_HDACT, P1 EXPANSION BUS, P9 TRAPDOOR, Q301 2N3906, Q321 MPF102, Q331 MPF102, Q501 2N3904, Q502 2N3906, Q503 2N3906, Q711 2N3904, Q921 MMBFJ113, Q931 MMBFJ113, Q99 2N3906, U1 68000D, U10 74LS244, U11 74LS373, U12 74LS244, U13 74LS373, U14 LF347, U15 74LS157, U16 XX4256, U17 XX4256, U18 XX4256, U19 XX4256, U2 FAT_AGNUS_8375, U20 XX4256, U21 XX4256, U22 XX4256, U23 XX4256, U3 PAULA, U32 74LS139, U33 74LS258, U34 74LS373, U35 74LS244, U36 74LS05, U37 74LS32, U38 MC1488, U39 MC1489, U4 DENISE, U40 74LS245, U41 74LS245, U42 NE555, U5 GARY_5719, U6 ROM, U7 VIA_8520, U8 VIA_8520, U9 MSM6242B, U90 DT1042, U91 DT1042, U92 DT1042, U93 DT1042, U94 74HCT14, X1 XTAL, Y9 32768

Commit message: updated rev 8A.2
Parts:
- removed U90, U91, U92, U93: DT1042, Raemixx500:TSOP-6_Handsolder
- added G***: LOGO, SBCLogoLargeLibrary:SBCLogoMiddle, F.Cu at (121.5, 211.8)
- moved G*** 56.4 mm to (355.8, 167.8)
Routing:
- net /Paula & Audio Stuff/potx2: track 55.1 -> 10.9 mm
- net /Paula & Audio Stuff/poty2: track 50.1 -> 15.1 mm
- net /Paula & Audio Stuff/vcc2: track 53.9 -> 23.0 mm
- net /Paula & Audio Stuff/right2: track 39.7 -> 11.0 mm
- net /Paula & Audio Stuff/fire1: track 72.7 -> 49.3 mm
- net /Paula & Audio Stuff/fire2: track 56.3 -> 34.4 mm
- net /Paula & Audio Stuff/left2: track 53.6 -> 31.8 mm
- net /Paula & Audio Stuff/down2: track 28.1 -> 8.84 mm
- net /Paula & Audio Stuff/up2: track 52.3 -> 34.6 mm
- net /Paula & Audio Stuff/vcc1: track 48.7 -> 31.0 mm
- net /Paula & Audio Stuff/up1: track 57.2 -> 42.1 mm
- net /Paula & Audio Stuff/poty1: track 37.3 -> 27.2 mm
- net /Paula & Audio Stuff/down1: track 57.0 -> 47.4 mm
- net /Paula & Audio Stuff/left1: track 24.0 -> 17.7 mm
- net /Paula & Audio Stuff/potx1: track 61.7 -> 55.9 mm
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Other:
- board text added: "A500++"
- board text removed: "A500sub"
