File: audio.kicad_sch (KiCad schematic)
At the start: 106 parts, among them CN1 LEFT_JOY, CN2 RIGHT_JOY, CN3 RIGHT, CN4 LEFT, Q301 2N3906, Q321 MPF102, Q331 MPF102, Q921 MMBFJ113, Q931 MMBFJ113, U14A LF347, U14B LF347, U14C LF347, U14D LF347, U14E LF347, U15A 74LS157, U15B 74LS157, U38A MC1488, U3A PAULA, U3B PAULA, U90 DT1042, U91 DT1042, U92 DT1042, U93 DT1042

Commit message: updated rev 8A.2
Parts:
- removed U90, U91, U92, U93: DT1042, Raemixx500:TSOP-6_Handsolder, symbol DT1042:DT1042
- renumbered U14A to U14A1, U14B to U14B1, U14C to U14C1, U14D to U14D1, U14E to U14E1, U15A to U15A1, U15B to U15B1, U38A to U38A1, U3A to U3A1, U3B to U3B1
Connections:
- no-connect marks 2 -> 0
Other:
- note removed: "EXTRA TVS DIODES FOR ESD PROTECTION"
- company: SukkoPera -> Submeson Brain Corperation
- title: Rämixx500 -> A500Sub
