File: cias.kicad_sch (KiCad schematic)
At the start: 78 parts, among them CN13 KEYBOARD, CN6 SERIAL_DB25M, CN7 PARALLEL_DB25F, J90 DRIVE_SWITCHER, J99 CONN_HDACT, Q501 2N3904, Q502 2N3906, Q503 2N3906, Q711 2N3904, Q99 2N3906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

Commit message: updated rev 8A.2
Parts:
- renumbered U38B to U38B1, U38C to U38C1, U38D to U38D1, U38E to U38E1, U39A to U39A1, U39B to U39B1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
Other:
- company: SukkoPera -> Submeson Brain Corperation
- title: Rämixx500 -> A500Sub
