File: clockdist.kicad_sch (KiCad schematic)
At the start: 19 parts, among them U33A 74LS258, U33B 74LS258, U33C 74LS258, U33E 74LS258

Commit message: updated rev 8A.2
Parts:
- renumbered U33A to U33A1, U33B to U33B1, U33C to U33C1, U33E to U33E1
Other:
- company: SukkoPera -> Submeson Brain Corperation
- title: Rämixx500 -> A500Sub
Changed lines of the file:
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@@
 	(paper "A4")
 	(title_block
-		(title "Rämixx500")
-		(date "2019-04-20")
-		(rev "1")
-		(company "SukkoPera")
-		(comment 4 "Licensed under CC BY-NC-SA 4.0")
+		(title "A500Sub")
+		(date "2026-01-06")
+		(rev "2")
+		(company "Submeson Brain Corperation")
 	)
 	(text "FCC GOOBERS"
@@
 				)
 			)
+			(project "clockdist"
+				(path "/4b1d4e11-b2b7-4a78-a363-402d7bcc9857"
+					(reference "E?")
+					(unit 1)
+				)
+			)
 		)
 	)
@@
 				)
 			)
+			(project "clockdist"
+				(path "/4b1d4e11-b2b7-4a78-a363-402d7bcc9857"
+					(reference "E?")
+					(unit 1)
+				)
+			)
 		)
 	)
@@
 				)
 			)
+			(project "clockdist"
+				(path "/4b1d4e11-b2b7-4a78-a363-402d7bcc9857"
+					(reference "E?")
+					(unit 1)
+				)
+			)
 		)
 	)
@@
 				)
 			)
+			(project "clockdist"
+				(path "/4b1d4e11-b2b7-4a78-a363-402d7bcc9857"
+					(reference "E?")
+					(unit 1)
+				)
+			)
 		)
 	)
@@
 				)
 			)
+			(project "clockdist"
+				(path "/4b1d4e11-b2b7-4a78-a363-402d7bcc9857"
+					(reference "E?")
+					(unit 1)
+				)
+			)
 		)
 	)
@@
 				)
 			)
+			(project "clockdist"
+				(path "/4b1d4e11-b2b7-4a78-a363-402d7bcc9857"
+					(reference "E?")
+					(unit 1)
+				)
+			)
 		)
 	)
@@
 				)
 			)
+			(project "clockdist"
+				(path "/4b1d4e11-b2b7-4a78-a363-402d7bcc9857"
+					(reference "E?")
+					(unit 1)
+				)
+			)
 		)
 	)
@@
 				)
 			)
+			(project "clockdist"
+				(path "/4b1d4e11-b2b7-4a78-a363-402d7bcc9857"
+					(reference "E?")
+					(unit 1)
+				)
+			)
 		)
 	)
@@
 				)
 			)
+			(project "clockdist"
+				(path "/4b1d4e11-b2b7-4a78-a363-402d7bcc9857"
+					(reference "#PWR?")
+					(unit 1)
+				)
+			)
 		)
 	)
@@
 				)
 			)
+			(project "clockdist"
+				(path "/4b1d4e11-b2b7-4a78-a363-402d7bcc9857"
+					(reference "#PWR?")
+					(unit 1)
+				)
+			)
 		)
 	)
@@
 				)
 			)
+			(project "clockdist"
+				(path "/4b1d4e11-b2b7-4a78-a363-402d7bcc9857"
+					(reference "E?")
+					(unit 1)
+				)
+			)
 		)
 	)
@@
 				)
 			)
+			(project "clockdist"
+				(path "/4b1d4e11-b2b7-4a78-a363-402d7bcc9857"
+					(reference "E?")
+					(unit 1)
+				)
+			)
 		)
 	)
@@
 				)
 			)
+			(project "clockdist"
+				(path "/4b1d4e11-b2b7-4a78-a363-402d7bcc9857"
+					(reference "#PWR?")
+					(unit 1)
+				)
+			)
 		)
 	)
@@
 				)
 			)
+			(project "clockdist"
+				(path "/4b1d4e11-b2b7-4a78-a363-402d7bcc9857"
+					(reference "E?")
+					(unit 1)
+				)
+			)
 		)
 	)
@@
 				)
 			)
+			(project "clockdist"
+				(path "/4b1d4e11-b2b7-4a78-a363-402d7bcc9857"
+					(reference "E?")
+					(unit 1)
+				)
+			)
 		)
 	)
@@
 		(on_board yes)
 		(dnp no)
-		(property "Reference" "U33A"
+		(property "Reference" "U33A1"
 			(at 93.726 60.96 0)
 			(effects
@@
 			(project "Raemixx500"
 				(path "/3fbeb09d-d0f9-4f56-b343-194274c97843/00000000-0000-0000-0000-00005d88ec26"
-					(reference "U33A")
+					(reference "U33A1")
+					(unit 1)
+				)
+			)
+			(project "clockdist"
+				(path "/4b1d4e11-b2b7-4a78-a363-402d7bcc9857"
+					(reference "U33A?")
 					(unit 1)
 				)
@@
 		(on_board yes)
 		(dnp no)
-		(property "Reference" "U33B"
+		(property "Reference" "U33B1"
 			(at 93.726 96.52 0)
 			(effects
@@
 			(project "Raemixx500"
 				(path "/3fbeb09d-d0f9-4f56-b343-194274c97843/00000000-0000-0000-0000-00005d88ec26"
-					(reference "U33B")
+					(reference "U33B1")
 					(unit 2)
 				)
 			)
+			(project "clockdist"
+				(path "/4b1d4e11-b2b7-4a78-a363-402d7bcc9857"
+					(reference "U33B?")
+					(unit 1)
+				)
+			)
 		)
 	)
@@
 		(on_board yes)
 		(dnp no)
-		(property "Reference" "U33C"
+		(property "Reference" "U33C1"
 			(at 93.726 78.74 0)
 			(effects
@@
 			(project "Raemixx500"
 				(path "/3fbeb09d-d0f9-4f56-b343-194274c97843/00000000-0000-0000-0000-00005d88ec26"
-					(reference "U33C")
+					(reference "U33C1")
 					(unit 3)
 				)
 			)
+			(project "clockdist"
+				(path "/4b1d4e11-b2b7-4a78-a363-402d7bcc9857"
+					(reference "U33C?")
+					(unit 1)
+				)
+			)
 		)
 	)
@@
 				)
 			)
+			(project "clockdist"
+				(path "/4b1d4e11-b2b7-4a78-a363-402d7bcc9857"
+					(reference "RP?")
+					(unit 1)
+				)
+			)
 		)
 	)
@@
 		(on_board yes)
 		(dnp no)
-		(property "Reference" "U33E"
+		(property "Reference" "U33E1"
 			(at 250.698 89.154 0)
 			(effects
@@
 			(project "Raemixx500"
 				(path "/3fbeb09d-d0f9-4f56-b343-194274c97843/00000000-0000-0000-0000-00005d88ec26"
-					(reference "U33E")
+					(reference "U33E1")
 					(unit 5)
 				)
 			)
+			(project "clockdist"
+				(path "/4b1d4e11-b2b7-4a78-a363-402d7bcc9857"
+					(reference "U33E?")
+					(unit 1)
+				)
+			)
 		)
 	)
@@
 				)
 			)
+			(project "clockdist"
+				(path "/4b1d4e11-b2b7-4a78-a363-402d7bcc9857"
+					(reference "#PWR?")
+					(unit 1)
+				)
+			)
 		)
 	)
@@
 				)
 			)
+			(project "clockdist"
+				(path "/4b1d4e11-b2b7-4a78-a363-402d7bcc9857"
+					(reference "#PWR?")
+					(unit 1)
+				)
+			)
 		)
 	)
@@
 				)
 			)
+			(project "clockdist"
+				(path "/4b1d4e11-b2b7-4a78-a363-402d7bcc9857"
+					(reference "#PWR?")
+					(unit 1)
+				)
+			)
 		)
 	)
@@
 				)
 			)
+			(project "clockdist"
+				(path "/4b1d4e11-b2b7-4a78-a363-402d7bcc9857"
+					(reference "E?")
+					(unit 1)
+				)
+			)
 		)
 	)
@@
 				)
 			)
+			(project "clockdist"
+				(path "/4b1d4e11-b2b7-4a78-a363-402d7bcc9857"
+					(reference "C?")
+					(unit 1)
+				)
+			)
+		)
+	)
+	(sheet_instances
+		(path "/"
+			(page "1")
 		)
 	)
+	(embedded_fonts no)
 )
