File: cpu.kicad_sch (KiCad schematic)
At the start: 27 parts, among them U10A 74LS244, U11A 74LS373, U12A 74LS244, U13A 74LS373, U1A 68000D, U2A FAT_AGNUS_8375, U33D 74LS258, U37A 74LS32, U37B 74LS32, U5A GARY_5719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

Commit message: updated rev 8A.2
Parts:
- renumbered U10A to U10A1, U11A to U11A1, U12A to U12A1, U13A to U13A1, U1A to U1A1, U2A to U2A1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
Other:
- company: SukkoPera -> Submeson Brain Corperation
- title: Rämixx500 -> A500Sub
