File: expansion.kicad_sch (KiCad schematic)
At the start: 4 parts, among them P1 EXPANSION BUS

Commit message: updated rev 8A.2
Other:
- company: SukkoPera -> Submeson Brain Corperation
- title: Rämixx500 -> A500Sub
Changed lines of the file:
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@@
 	(paper "A4")
 	(title_block
-		(title "Rämixx500")
-		(date "2019-06-23")
-		(rev "1")
-		(company "SukkoPera")
-		(comment 4 "Licensed under CC BY-NC-SA 4.0")
+		(title "A500Sub")
+		(date "2026-01-06")
+		(rev "2")
+		(company "Submeson Brain Corperation")
 	)
 	(junction
@@
 				)
 			)
+			(project "expansion"
+				(path "/f141b82a-951c-4742-a2a2-aff557813c39"
+					(reference "P?")
+					(unit 1)
+				)
+			)
 		)
 	)
@@
 				)
 			)
+			(project "expansion"
+				(path "/f141b82a-951c-4742-a2a2-aff557813c39"
+					(reference "#PWR?")
+					(unit 1)
+				)
+			)
 		)
 	)
@@
 				)
 			)
+			(project "expansion"
+				(path "/f141b82a-951c-4742-a2a2-aff557813c39"
+					(reference "#PWR?")
+					(unit 1)
+				)
+			)
 		)
 	)
@@
 				)
 			)
+			(project "expansion"
+				(path "/f141b82a-951c-4742-a2a2-aff557813c39"
+					(reference "E?")
+					(unit 1)
+				)
+			)
 		)
 	)
@@
 				)
 			)
+			(project "expansion"
+				(path "/f141b82a-951c-4742-a2a2-aff557813c39"
+					(reference "E?")
+					(unit 1)
+				)
+			)
 		)
 	)
@@
 				)
 			)
+			(project "expansion"
+				(path "/f141b82a-951c-4742-a2a2-aff557813c39"
+					(reference "E?")
+					(unit 1)
+				)
+			)
 		)
 	)
@@
 				)
 			)
+			(project "expansion"
+				(path "/f141b82a-951c-4742-a2a2-aff557813c39"
+					(reference "#PWR?")
+					(unit 1)
+				)
+			)
 		)
 	)
@@
 				)
 			)
+			(project "expansion"
+				(path "/f141b82a-951c-4742-a2a2-aff557813c39"
+					(reference "#PWR?")
+					(unit 1)
+				)
+			)
 		)
 	)
@@
 				)
 			)
+			(project "expansion"
+				(path "/f141b82a-951c-4742-a2a2-aff557813c39"
+					(reference "#PWR?")
+					(unit 1)
+				)
+			)
+		)
+	)
+	(sheet_instances
+		(path "/"
+			(page "1")
 		)
 	)
+	(embedded_fonts no)
 )
