File: floppy.kicad_sch (KiCad schematic)
At the start: 28 parts, among them CN11 INTERNAL_FLOPPY, CN12 FLOPPY_POWER, CN14 IDE_POWER, CN15 IDE_I/F, CN5 EXTFLOPPY_DB23F, U36A 74LS05, U36B 74LS05, U36C 74LS05, U36D 74LS05, U5B GARY_5719

Commit message: updated rev 8A.2
Parts:
- renumbered U36A to U36A1, U36B to U36B1, U36C to U36C1, U36D to U36D1, U5B to U5B1
Other:
- company: SukkoPera -> Submeson Brain Corperation
- title: Rämixx500 -> A500Sub
