File: power.kicad_sch (KiCad schematic)
At the start: 51 parts, among them CN8 POWER, U10B 74LS244, U11B 74LS373, U12B 74LS244, U13B 74LS373, U1B 68000D, U2B FAT_AGNUS_8375, U32C 74LS139, U34B 74LS373, U35B 74LS244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

Commit message: updated rev 8A.2
Parts:
- renumbered U10B to U10B1, U11B to U11B1, U12B to U12B1, U13B to U13B1, U1B to U1B1, U2B to U2B1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
Other:
- company: SukkoPera -> Submeson Brain Corperation
- title: Rämixx500 -> A500Sub
