File: ram.kicad_sch (KiCad schematic)
At the start: 34 parts, among them U16A XX4256, U16B XX4256, U17A XX4256, U17B XX4256, U18A XX4256, U18B XX4256, U19A XX4256, U19B XX4256, U20A XX4256, U20B XX4256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

Commit message: updated rev 8A.2
Parts:
- renumbered U16A to U16A1, U16B to U16B1, U17A to U17A1, U17B to U17B1, U18A to U18A1, U18B to U18B1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
Other:
- company: SukkoPera -> Submeson Brain Corperation
- title: Rämixx500 -> A500Sub
