File: rom.kicad_sch (KiCad schematic)
At the start: 6 parts, among them J91 Dispatcher_3to1, J92 Dispatcher_3to1, J93 Dispatcher_3to1, U6A ROM, U6B ROM

Commit message: updated rev 8A.2
Parts:
- renumbered U6A to U6A1, U6B to U6B1
Other:
- company: SukkoPera -> Submeson Brain Corperation
- title: Rämixx500 -> A500Sub
Changed lines of the file:
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@@
 	(paper "A4")
 	(title_block
-		(title "Rämixx500")
-		(date "2019-04-20")
-		(rev "1")
-		(company "SukkoPera")
-		(comment 4 "Licensed under CC BY-NC-SA 4.0")
+		(title "A500Sub")
+		(date "2026-01-06")
+		(rev "2")
+		(company "Submeson Brain Corperation")
 	)
 	(text "Simple Kickstart switcher, allowing\narbitrary driving of the high ROM\naddress lines. With a 27C160 EPROM,\nup to 8x256K Kickstart images can\nbe selected."
@@
 		(on_board yes)
 		(dnp no)
-		(property "Reference" "U6A"
+		(property "Reference" "U6A1"
 			(at 168.656 56.642 0)
 			(effects
@@
 			(project "Raemixx500"
 				(path "/3fbeb09d-d0f9-4f56-b343-194274c97843/00000000-0000-0000-0000-00005d86dd46"
-					(reference "U6A")
+					(reference "U6A1")
+					(unit 1)
+				)
+			)
+			(project "rom"
+				(path "/74164df9-a8b8-405e-9a14-f9bf6770489b"
+					(reference "U6A?")
 					(unit 1)
 				)
@@
 				)
 			)
+			(project "rom"
+				(path "/74164df9-a8b8-405e-9a14-f9bf6770489b"
+					(reference "#PWR?")
+					(unit 1)
+				)
+			)
 		)
 	)
@@
 				)
 			)
+			(project "rom"
+				(path "/74164df9-a8b8-405e-9a14-f9bf6770489b"
+					(reference "#PWR?")
+					(unit 1)
+				)
+			)
 		)
 	)
@@
 		(on_board yes)
 		(dnp no)
-		(property "Reference" "U6B"
+		(property "Reference" "U6B1"
 			(at 250.1392 89.5096 0)
 			(effects
@@
 			(project "Raemixx500"
 				(path "/3fbeb09d-d0f9-4f56-b343-194274c97843/00000000-0000-0000-0000-00005d86dd46"
-					(reference "U6B")
+					(reference "U6B1")
 					(unit 2)
 				)
 			)
+			(project "rom"
+				(path "/74164df9-a8b8-405e-9a14-f9bf6770489b"
+					(reference "U6B?")
+					(unit 1)
+				)
+			)
 		)
 	)
@@
 				)
 			)
+			(project "rom"
+				(path "/74164df9-a8b8-405e-9a14-f9bf6770489b"
+					(reference "#PWR?")
+					(unit 1)
+				)
+			)
 		)
 	)
@@
 				)
 			)
+			(project "rom"
+				(path "/74164df9-a8b8-405e-9a14-f9bf6770489b"
+					(reference "#PWR?")
+					(unit 1)
+				)
+			)
 		)
 	)
@@
 				)
 			)
+			(project "rom"
+				(path "/74164df9-a8b8-405e-9a14-f9bf6770489b"
+					(reference "C?")
+					(unit 1)
+				)
+			)
 		)
 	)
@@
 				)
 			)
+			(project "rom"
+				(path "/74164df9-a8b8-405e-9a14-f9bf6770489b"
+					(reference "#PWR?")
+					(unit 1)
+				)
+			)
 		)
 	)
@@
 				)
 			)
+			(project "rom"
+				(path "/74164df9-a8b8-405e-9a14-f9bf6770489b"
+					(reference "#PWR?")
+					(unit 1)
+				)
+			)
 		)
 	)
@@
 				)
 			)
+			(project "rom"
+				(path "/74164df9-a8b8-405e-9a14-f9bf6770489b"
+					(reference "J?")
+					(unit 1)
+				)
+			)
 		)
 	)
@@
 				)
 			)
+			(project "rom"
+				(path "/74164df9-a8b8-405e-9a14-f9bf6770489b"
+					(reference "#PWR?")
+					(unit 1)
+				)
+			)
 		)
 	)
@@
 				)
 			)
+			(project "rom"
+				(path "/74164df9-a8b8-405e-9a14-f9bf6770489b"
+					(reference "#PWR?")
+					(unit 1)
+				)
+			)
 		)
 	)
@@
 				)
 			)
+			(project "rom"
+				(path "/74164df9-a8b8-405e-9a14-f9bf6770489b"
+					(reference "J?")
+					(unit 1)
+				)
+			)
 		)
 	)
@@
 				)
 			)
+			(project "rom"
+				(path "/74164df9-a8b8-405e-9a14-f9bf6770489b"
+					(reference "#PWR?")
+					(unit 1)
+				)
+			)
 		)
 	)
@@
 				)
 			)
+			(project "rom"
+				(path "/74164df9-a8b8-405e-9a14-f9bf6770489b"
+					(reference "#PWR?")
+					(unit 1)
+				)
+			)
 		)
 	)
@@
 				)
 			)
+			(project "rom"
+				(path "/74164df9-a8b8-405e-9a14-f9bf6770489b"
+					(reference "J?")
+					(unit 1)
+				)
+			)
+		)
+	)
+	(sheet_instances
+		(path "/"
+			(page "1")
 		)
 	)
+	(embedded_fonts no)
 )
