File: rtc.kicad_sch (KiCad schematic)
At the start: 18 parts, among them U36E 74LS05, U36F 74LS05, U9A MSM6242B, U9B MSM6242B, Y9 32768

Commit message: updated rev 8A.2
Parts:
- renumbered U36E to U36E1, U36F to U36F1, U9A to U9A1, U9B to U9B1
Other:
- company: SukkoPera -> Submeson Brain Corperation
- title: Rämixx500 -> A500Sub
Changed lines of the file:
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@@
 	(paper "A4")
 	(title_block
-		(title "Rämixx500")
-		(date "2021-05-23")
-		(rev "1")
-		(company "SukkoPera")
-		(comment 4 "Licensed under CC BY-NC-SA 4.0")
+		(title "A500Sub")
+		(date "2026-01-06")
+		(rev "2")
+		(company "Submeson Brain Corperation")
 	)
 	(text "This diode is not installed in its place on original boards,\nas its cathode would connect to the other side or the\nresistor. But we'll fix this, so please install it normally."
@@
 		(on_board yes)
 		(dnp no)
-		(property "Reference" "U9A"
+		(property "Reference" "U9A1"
 			(at 203.073 34.544 0)
 			(effects
@@
 			(project "Raemixx500"
 				(path "/3fbeb09d-d0f9-4f56-b343-194274c97843/00000000-0000-0000-0000-00005cf615ab"
-					(reference "U9A")
+					(reference "U9A1")
+					(unit 1)
+				)
+			)
+			(project "rtc"
+				(path "/fcc4bb46-9321-4578-981a-1a5fc264cf5d"
+					(reference "U9A?")
 					(unit 1)
 				)
@@
 		(on_board yes)
 		(dnp no)
-		(property "Reference" "U36E"
+		(property "Reference" "U36E1"
 			(at 118.11 64.135 0)
 			(effects
@@
 			(project "Raemixx500"
 				(path "/3fbeb09d-d0f9-4f56-b343-194274c97843/00000000-0000-0000-0000-00005cf615ab"
-					(reference "U36E")
+					(reference "U36E1")
 					(unit 5)
 				)
 			)
+			(project "rtc"
+				(path "/fcc4bb46-9321-4578-981a-1a5fc264cf5d"
+					(reference "U36E?")
+					(unit 1)
+				)
+			)
 		)
 	)
@@
 				)
 			)
+			(project "rtc"
+				(path "/fcc4bb46-9321-4578-981a-1a5fc264cf5d"
+					(reference "R?")
+					(unit 1)
+				)
+			)
 		)
 	)
@@
 				)
 			)
+			(project "rtc"
+				(path "/fcc4bb46-9321-4578-981a-1a5fc264cf5d"
+					(reference "#PWR?")
+					(unit 1)
+				)
+			)
 		)
 	)
@@
 				)
 			)
+			(project "rtc"
+				(path "/fcc4bb46-9321-4578-981a-1a5fc264cf5d"
+					(reference "R?")
+					(unit 1)
+				)
+			)
 		)
 	)
@@
 				)
 			)
+			(project "rtc"
+				(path "/fcc4bb46-9321-4578-981a-1a5fc264cf5d"
+					(reference "R?")
+					(unit 1)
+				)
+			)
 		)
 	)
@@
 				)
 			)
+			(project "rtc"
+				(path "/fcc4bb46-9321-4578-981a-1a5fc264cf5d"
+					(reference "JP?")
+					(unit 1)
+				)
+			)
 		)
 	)
@@
 				)
 			)
+			(project "rtc"
+				(path "/fcc4bb46-9321-4578-981a-1a5fc264cf5d"
+					(reference "#PWR?")
+					(unit 1)
+				)
+			)
 		)
 	)
@@
 				)
 			)
+			(project "rtc"
+				(path "/fcc4bb46-9321-4578-981a-1a5fc264cf5d"
+					(reference "TC?")
+					(unit 1)
+				)
+			)
 		)
 	)
@@
 				)
 			)
+			(project "rtc"
+				(path "/fcc4bb46-9321-4578-981a-1a5fc264cf5d"
+					(reference "C?")
+					(unit 1)
+				)
+			)
 		)
 	)
@@
 				)
 			)
+			(project "rtc"
+				(path "/fcc4bb46-9321-4578-981a-1a5fc264cf5d"
+					(reference "#PWR?")
+					(unit 1)
+				)
+			)
 		)
 	)
@@
 		(on_board yes)
 		(dnp no)
-		(property "Reference" "U36F"
+		(property "Reference" "U36F1"
 			(at 79.629 64.135 0)
 			(effects
@@
 			(project "Raemixx500"
 				(path "/3fbeb09d-d0f9-4f56-b343-194274c97843/00000000-0000-0000-0000-00005cf615ab"
-					(reference "U36F")
+					(reference "U36F1")
 					(unit 6)
 				)
 			)
+			(project "rtc"
+				(path "/fcc4bb46-9321-4578-981a-1a5fc264cf5d"
+					(reference "U36F?")
+					(unit 1)
+				)
+			)
 		)
 	)
@@
 				)
 			)
+			(project "rtc"
+				(path "/fcc4bb46-9321-4578-981a-1a5fc264cf5d"
+					(reference "Y?")
+					(unit 1)
+				)
+			)
 		)
 	)
@@
 				)
 			)
+			(project "rtc"
+				(path "/fcc4bb46-9321-4578-981a-1a5fc264cf5d"
+					(reference "BT?")
+					(unit 1)
+				)
+			)
 		)
 	)
@@
 				)
 			)
+			(project "rtc"
+				(path "/fcc4bb46-9321-4578-981a-1a5fc264cf5d"
+					(reference "C?")
+					(unit 1)
+				)
+			)
 		)
 	)
@@
 		(on_board yes)
 		(dnp no)
-		(property "Reference" "U9B"
+		(property "Reference" "U9B1"
 			(at 122.7582 146.7866 0)
 			(effects
@@
 			(project "Raemixx500"
 				(path "/3fbeb09d-d0f9-4f56-b343-194274c97843/00000000-0000-0000-0000-00005cf615ab"
-					(reference "U9B")
+					(reference "U9B1")
 					(unit 2)
 				)
 			)
+			(project "rtc"
+				(path "/fcc4bb46-9321-4578-981a-1a5fc264cf5d"
+					(reference "U9B?")
+					(unit 1)
+				)
+			)
 		)
 	)
@@
 				)
 			)
+			(project "rtc"
+				(path "/fcc4bb46-9321-4578-981a-1a5fc264cf5d"
+					(reference "C?")
+					(unit 1)
+				)
+			)
 		)
 	)
@@
 				)
 			)
+			(project "rtc"
+				(path "/fcc4bb46-9321-4578-981a-1a5fc264cf5d"
+					(reference "#PWR?")
+					(unit 1)
+				)
+			)
 		)
 	)
@@
 				)
 			)
+			(project "rtc"
+				(path "/fcc4bb46-9321-4578-981a-1a5fc264cf5d"
+					(reference "D?")
+					(unit 1)
+				)
+			)
 		)
 	)
@@
 				)
 			)
+			(project "rtc"
+				(path "/fcc4bb46-9321-4578-981a-1a5fc264cf5d"
+					(reference "D?")
+					(unit 1)
+				)
+			)
 		)
 	)
@@
 				)
 			)
+			(project "rtc"
+				(path "/fcc4bb46-9321-4578-981a-1a5fc264cf5d"
+					(reference "R?")
+					(unit 1)
+				)
+			)
 		)
 	)
@@
 				)
 			)
+			(project "rtc"
+				(path "/fcc4bb46-9321-4578-981a-1a5fc264cf5d"
+					(reference "#PWR?")
+					(unit 1)
+				)
+			)
 		)
 	)
@@
 				)
 			)
+			(project "rtc"
+				(path "/fcc4bb46-9321-4578-981a-1a5fc264cf5d"
+					(reference "#PWR?")
+					(unit 1)
+				)
+			)
 		)
 	)
@@
 				)
 			)
+			(project "rtc"
+				(path "/fcc4bb46-9321-4578-981a-1a5fc264cf5d"
+					(reference "D?")
+					(unit 1)
+				)
+			)
+		)
+	)
+	(sheet_instances
+		(path "/"
+			(page "1")
 		)
 	)
+	(embedded_fonts no)
 )
