File: terminators.kicad_sch (KiCad schematic)
At the start: 14 parts, among them U37C 74LS32, U37D 74LS32

Commit message: updated rev 8A.2
Parts:
- renumbered U37C to U37C1, U37D to U37D1
Other:
- company: SukkoPera -> Submeson Brain Corperation
- title: Rämixx500 -> 500ub
Changed lines of the file:
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@@
 	(paper "A4")
 	(title_block
-		(title "Rämixx500")
-		(date "2021-05-16")
-		(rev "1")
-		(company "SukkoPera")
-		(comment 4 "Licensed under CC BY-NC-SA 4.0")
+		(title "500ub")
+		(date "2026-01-06")
+		(rev "2")
+		(company "Submeson Brain Corperation")
 	)
 	(text "Note: RP105-RP111 are optional internal bus\ntermination, and are not normally loaded."
@@
 				)
 			)
+			(project "terminators"
+				(path "/4383d6a1-8db7-4289-9495-6f46c0eb3cd0"
+					(reference "RP?")
+					(unit 1)
+				)
+			)
 		)
 	)
@@
 				)
 			)
+			(project "terminators"
+				(path "/4383d6a1-8db7-4289-9495-6f46c0eb3cd0"
+					(reference "RP?")
+					(unit 1)
+				)
+			)
 		)
 	)
@@
 				)
 			)
+			(project "terminators"
+				(path "/4383d6a1-8db7-4289-9495-6f46c0eb3cd0"
+					(reference "RP?")
+					(unit 1)
+				)
+			)
 		)
 	)
@@
 				)
 			)
+			(project "terminators"
+				(path "/4383d6a1-8db7-4289-9495-6f46c0eb3cd0"
+					(reference "#PWR?")
+					(unit 1)
+				)
+			)
 		)
 	)
@@
 				)
 			)
+			(project "terminators"
+				(path "/4383d6a1-8db7-4289-9495-6f46c0eb3cd0"
+					(reference "#PWR?")
+					(unit 1)
+				)
+			)
 		)
 	)
@@
 				)
 			)
+			(project "terminators"
+				(path "/4383d6a1-8db7-4289-9495-6f46c0eb3cd0"
+					(reference "RP?")
+					(unit 1)
+				)
+			)
 		)
 	)
@@
 				)
 			)
+			(project "terminators"
+				(path "/4383d6a1-8db7-4289-9495-6f46c0eb3cd0"
+					(reference "RP?")
+					(unit 1)
+				)
+			)
 		)
 	)
@@
 				)
 			)
+			(project "terminators"
+				(path "/4383d6a1-8db7-4289-9495-6f46c0eb3cd0"
+					(reference "#PWR?")
+					(unit 1)
+				)
+			)
 		)
 	)
@@
 				)
 			)
+			(project "terminators"
+				(path "/4383d6a1-8db7-4289-9495-6f46c0eb3cd0"
+					(reference "#PWR?")
+					(unit 1)
+				)
+			)
 		)
 	)
@@
 				)
 			)
+			(project "terminators"
+				(path "/4383d6a1-8db7-4289-9495-6f46c0eb3cd0"
+					(reference "RP?")
+					(unit 1)
+				)
+			)
 		)
 	)
@@
 				)
 			)
+			(project "terminators"
+				(path "/4383d6a1-8db7-4289-9495-6f46c0eb3cd0"
+					(reference "RP?")
+					(unit 1)
+				)
+			)
 		)
 	)
@@
 				)
 			)
+			(project "terminators"
+				(path "/4383d6a1-8db7-4289-9495-6f46c0eb3cd0"
+					(reference "#PWR?")
+					(unit 1)
+				)
+			)
 		)
 	)
@@
 				)
 			)
+			(project "terminators"
+				(path "/4383d6a1-8db7-4289-9495-6f46c0eb3cd0"
+					(reference "#PWR?")
+					(unit 1)
+				)
+			)
 		)
 	)
@@
 				)
 			)
+			(project "terminators"
+				(path "/4383d6a1-8db7-4289-9495-6f46c0eb3cd0"
+					(reference "RP?")
+					(unit 1)
+				)
+			)
 		)
 	)
@@
 				)
 			)
+			(project "terminators"
+				(path "/4383d6a1-8db7-4289-9495-6f46c0eb3cd0"
+					(reference "#PWR?")
+					(unit 1)
+				)
+			)
 		)
 	)
@@
 				)
 			)
+			(project "terminators"
+				(path "/4383d6a1-8db7-4289-9495-6f46c0eb3cd0"
+					(reference "#PWR?")
+					(unit 1)
+				)
+			)
 		)
 	)
@@
 				)
 			)
+			(project "terminators"
+				(path "/4383d6a1-8db7-4289-9495-6f46c0eb3cd0"
+					(reference "#PWR?")
+					(unit 1)
+				)
+			)
 		)
 	)
@@
 				)
 			)
+			(project "terminators"
+				(path "/4383d6a1-8db7-4289-9495-6f46c0eb3cd0"
+					(reference "R?")
+					(unit 1)
+				)
+			)
 		)
 	)
@@
 				)
 			)
+			(project "terminators"
+				(path "/4383d6a1-8db7-4289-9495-6f46c0eb3cd0"
+					(reference "R?")
+					(unit 1)
+				)
+			)
 		)
 	)
@@
 				)
 			)
+			(project "terminators"
+				(path "/4383d6a1-8db7-4289-9495-6f46c0eb3cd0"
+					(reference "RP?")
+					(unit 1)
+				)
+			)
 		)
 	)
@@
 				)
 			)
+			(project "terminators"
+				(path "/4383d6a1-8db7-4289-9495-6f46c0eb3cd0"
+					(reference "RP?")
+					(unit 1)
+				)
+			)
 		)
 	)
@@
 				)
 			)
+			(project "terminators"
+				(path "/4383d6a1-8db7-4289-9495-6f46c0eb3cd0"
+					(reference "#PWR?")
+					(unit 1)
+				)
+			)
 		)
 	)
@@
 				)
 			)
+			(project "terminators"
+				(path "/4383d6a1-8db7-4289-9495-6f46c0eb3cd0"
+					(reference "#PWR?")
+					(unit 1)
+				)
+			)
 		)
 	)
@@
 		(on_board yes)
 		(dnp no)
-		(property "Reference" "U37D"
+		(property "Reference" "U37D1"
 			(at 219.964 123.952 0)
 			(effects
@@
 			(project "Raemixx500"
 				(path "/3fbeb09d-d0f9-4f56-b343-194274c97843/00000000-0000-0000-0000-00005d6d5ebe"
-					(reference "U37D")
+					(reference "U37D1")
 					(unit 4)
 				)
 			)
+			(project "terminators"
+				(path "/4383d6a1-8db7-4289-9495-6f46c0eb3cd0"
+					(reference "U37D?")
+					(unit 1)
+				)
+			)
 		)
 	)
@@
 		(on_board yes)
 		(dnp no)
-		(property "Reference" "U37C"
+		(property "Reference" "U37C1"
 			(at 244.475 136.017 0)
 			(effects
@@
 			(project "Raemixx500"
 				(path "/3fbeb09d-d0f9-4f56-b343-194274c97843/00000000-0000-0000-0000-00005d6d5ebe"
-					(reference "U37C")
+					(reference "U37C1")
 					(unit 3)
 				)
 			)
+			(project "terminators"
+				(path "/4383d6a1-8db7-4289-9495-6f46c0eb3cd0"
+					(reference "U37C?")
+					(unit 1)
+				)
+			)
 		)
 	)
@@
 				)
 			)
+			(project "terminators"
+				(path "/4383d6a1-8db7-4289-9495-6f46c0eb3cd0"
+					(reference "#PWR?")
+					(unit 1)
+				)
+			)
+		)
+	)
+	(sheet_instances
+		(path "/"
+			(page "1")
 		)
 	)
+	(embedded_fonts no)
 )
