File: trapdoor.kicad_sch (KiCad schematic)
At the start: 2 parts, among them P9 TRAPDOOR

Commit message: updated rev 8A.2
Other:
- company: SukkoPera -> Submeson Brain Corperation
- title: Rämixx500 -> A500Sub
Changed lines of the file:
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@@
 	(paper "A4")
 	(title_block
-		(title "Rämixx500")
-		(date "2020-04-05")
-		(rev "1")
-		(company "SukkoPera")
-		(comment 4 "Licensed under CC BY-NC-SA 4.0")
+		(title "A500Sub")
+		(date "2026-01-06")
+		(rev "2")
+		(company "Submeson Brain Corperation")
 	)
 	(junction
@@
 				)
 			)
+			(project "trapdoor"
+				(path "/e59f2b38-25b4-40fe-b3fd-a2ef5aca637d"
+					(reference "P?")
+					(unit 1)
+				)
+			)
 		)
 	)
@@
 				)
 				(path "/3fbeb09d-d0f9-4f56-b343-194274c97843/00000000-0000-0000-0000-00005e813dc5"
+					(reference "#PWR?")
+					(unit 1)
+				)
+			)
+			(project "trapdoor"
+				(path "/e59f2b38-25b4-40fe-b3fd-a2ef5aca637d"
 					(reference "#PWR?")
 					(unit 1)
@@
 				)
 			)
+			(project "trapdoor"
+				(path "/e59f2b38-25b4-40fe-b3fd-a2ef5aca637d"
+					(reference "#PWR?")
+					(unit 1)
+				)
+			)
 		)
 	)
@@
 				(path "/3fbeb09d-d0f9-4f56-b343-194274c97843/00000000-0000-0000-0000-00005d00c589"
 					(reference "#PWR0254")
+					(unit 1)
+				)
+			)
+			(project "trapdoor"
+				(path "/e59f2b38-25b4-40fe-b3fd-a2ef5aca637d"
+					(reference "#PWR?")
 					(unit 1)
 				)
@@
 				)
 			)
+			(project "trapdoor"
+				(path "/e59f2b38-25b4-40fe-b3fd-a2ef5aca637d"
+					(reference "#PWR?")
+					(unit 1)
+				)
+			)
 		)
 	)
@@
 				(path "/3fbeb09d-d0f9-4f56-b343-194274c97843/00000000-0000-0000-0000-00005d00c589"
 					(reference "#PWR0256")
+					(unit 1)
+				)
+			)
+			(project "trapdoor"
+				(path "/e59f2b38-25b4-40fe-b3fd-a2ef5aca637d"
+					(reference "#PWR?")
 					(unit 1)
 				)
@@
 				)
 			)
+			(project "trapdoor"
+				(path "/e59f2b38-25b4-40fe-b3fd-a2ef5aca637d"
+					(reference "#PWR?")
+					(unit 1)
+				)
+			)
 		)
 	)
@@
 				)
 			)
-		)
-	)
+			(project "trapdoor"
+				(path "/e59f2b38-25b4-40fe-b3fd-a2ef5aca637d"
+					(reference "JP7A?")
+					(unit 1)
+				)
+			)
+		)
+	)
+	(sheet_instances
+		(path "/"
+			(page "1")
+		)
+	)
+	(embedded_fonts no)
 )
