File: video.kicad_sch (KiCad schematic)
At the start: 46 parts, among them CN10 COMPOSITE, CN9 VIDEO_DB23M, U40A 74LS245, U40B 74LS245, U41A 74LS245, U41B 74LS245, U4A DENISE, U4B DENISE, U94A 74HCT14, U94B 74HCT14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

Commit message: updated rev 8A.2
Parts:
- renumbered HY1A to HY1A1, HY1B to HY1B1, U40A to U40A1, U40B to U40B1, U41A to U41A1, U41B to U41B1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
Other:
- company: SukkoPera -> Submeson Brain Corperation
- title: Rämixx500 -> A500Sub
