File: src/Amiga500.kicad_pcb (KiCad board)
At the start: 2 copper layers, 365.8 x 254 mm, 367 parts, among them CN1 LEFT_JOY, CN10 COMPOSITE, CN11 INTERNAL_FLOPPY, CN12 FLOPPY_POWER, CN13 KEYBOARD, CN14 IDE_POWER, CN15 IDE_I/F, CN2 RIGHT_JOY, CN3 RIGHT, CN4 LEFT, CN5 EXTFLOPPY_DB23F, CN6 SERIAL_DB25M, CN7 PARALLEL_DB25F, CN8 POWER, CN9 VIDEO_DB23M, J90 DRIVE_SWITCHER, J91 Dispatcher_3to1, J92 Dispatcher_3to1, J93 Dispatcher_3to1, J99 CONN_HDACT, P1 EXPANSION BUS, P9 TRAPDOOR, Q301 2N3906, Q321 MPF102, Q331 MPF102, Q501 2N3904, Q502 2N3906, Q503 2N3906, Q711 2N3904, Q921 MMBFJ113, Q931 MMBFJ113, Q99 2N3906, U1 68000D, U10 74LS244, U11 74LS373, U12 74LS244, U13 74LS373, U14 LF347, U15 74LS157, U16 XX4256, U17 XX4256, U18 XX4256, U19 XX4256, U2 FAT_AGNUS_8375, U20 XX4256, U21 XX4256, U22 XX4256, U23 XX4256, U3 PAULA, U32 74LS139, U33 74LS258, U34 74LS373, U35 74LS244, U36 74LS05, U37 74LS32, U38 MC1488, U39 MC1489, U4 DENISE, U40 74LS245, U41 74LS245, U42 NE555, U5 GARY_5719, U6 ROM, U7 VIA_8520, U8 VIA_8520, U9 MSM6242B, U94 74HCT14, X1 XTAL, Y9 32768

Commit message: Added 3D models
Parts:
- removed the G*** at (121.5, 211.8)
- added G***: LOGO, Commodore Logo:Commodore Logo Outlined little, F.Cu at (121.8, 211.7)
- moved G*** 54.9 mm to (356.5, 112.8)
Other:
- board text added: "+"
- board text added: "A recreation of the Commodore Amiga A500+ with a few enhancements Created by Bambleweeny57 for the Submeson Brain Corporation (a playful tribute to Commodore and Douglas Adams)"
- board text added: "A500"
- board text added: "A500+"
- board text removed: "A500++"
- board text removed: "TOGETHER WE STAND, DIVIDED WE FALL"
