File: src/audio.kicad_sch (KiCad schematic)
At the start: 102 parts, among them CN1 LEFT_JOY, CN2 RIGHT_JOY, CN3 RIGHT, CN4 LEFT, Q301 2N3906, Q321 MPF102, Q331 MPF102, Q921 MMBFJ113, Q931 MMBFJ113, U14A1 LF347, U14B1 LF347, U14C1 LF347, U14D1 LF347, U14E1 LF347, U15A1 74LS157, U15B1 74LS157, U38A1 MC1488, U3A1 PAULA, U3B1 PAULA

Commit message: changed silkscreen thickness
Parts:
- renumbered C411 to C?, C413 to C?, C412 to C?, C421 to C?, C423 to C?, C422 to C?, C3 to C?, C307 to C?, C312 to C?, C311 to C?, C314 to C?, C313 to C?, C321 to C?, C322 to C?, C325 to C?, C324 to C?, C305 to C?, C306 to C?, C301 to C?, C303 to C?, C302 to C?, C304 to C?, C331 to C?, C332 to C?, C335 to C?, C334 to C?, C323 to C?, C333 to C?, C308 to C?, C15 to C?, CN1 to CN?, CN2 to CN?, CN3 to CN?, CN4 to CN?, E415 to E?, E401 to E?, E416 to E?, E417 to E?, E425 to E?, E408 to E?, E426 to E?, E427 to E?, E411 to E?, E412 to E?, E413 to E?, E414 to E?, E421 to E?, E422 to E?, E423 to E?, E424 to E?, E441 to E?, E443 to E?, E444 to E?, E442 to E?, E305 to E?, E306 to E?, E302 to E?, E303 to E?, FB802 to FB?, JP10A1 to JP10A?, JP10B1 to JP10B?, JP8 to JP?, Q321 to Q?, Q331 to Q?, Q301 to Q?, Q931 to Q?, Q921 to Q?, R401 to R?, R408 to R?, R309 to R?, R303 to R?, R321 to R?, R322 to R?, R323 to R?, R304 to R?, R324 to R?, R325 to R?, R301 to R?, R302 to R?, R326 to R?, R331 to R?, R332 to R?, R333 to R?, R334 to R?, R335 to R?, R336 to R?, R308 to R?, R306 to R?, R305 to R?, R307 to R?, R339 to R?, RP401 to RP?, U14A1 to U14A?, U14B1 to U14B?, U14C1 to U14C?, U14D1 to U14D?, U14E1 to U14E?, U15A1 to U15A?, U15B1 to U15B?, U38A1 to U38A?, U3A1 to U3A?, U3B1 to U3B?
Connections:
- net +VDC: no longer U14E?.4 (V+)
- net -VDC: no longer U14E?.11 (V-)
- net GND: no longer U15B?.8 (GND), U3B?.8 (GND)
- net VAC: now also U14C?.3 (+), U14D?.3 (+); no longer U14C?.10 (+), U14D?.12 (+)
- net VCC: no longer U15B?.16 (VCC)
- net at C?.1, C?.1, R?.2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: no longer U3B?.27 (VCC)
- net at C?.1, Q?.2 (S), Q?.2 (S)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: now also U14B?.3 (+); no longer U14B?.5 (+)
- net at C?.1, C?.1, C?.2: now also U14B?.1, U14B?.2 (-); no longer U14B?.6 (-), U14B?.7
- net at C?.1, Q?.1 (D), Q?.1 (D)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: now also U14C?.1; no longer U14C?.8
- net at C?.2, E?.3, R?.1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: now also U14C?.2 (-); no longer U14C?.9 (-)
- net at C?.2, E?.3, R?.2: now also U14D?.2 (-); no longer U14D?.13 (-)
- net at C?.1, Q?.1 (D), Q?.1 (D)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: now also U14D?.1; no longer U14D?.14
