File: src/audio.kicad_sch (KiCad schematic)
At the start: 102 parts, among them U14A? LF347, U14B? LF347, U14C? LF347, U14D? LF347, U14E? LF347, U15A? 74LS157, U15B? 74LS157, U38A? MC1488, U3A? PAULA, U3B? PAULA

Commit message: kicad 10
Parts:
- gave numbers to parts that had none: 102
Connections:
- net +VDC: now also U14E1.4 (V+)
- net -VDC: now also U14E1.11 (V-)
- net GND: now also U15B1.8 (GND), U3B1.8 (GND)
- net VAC: now also U14C1.10 (+), U14D1.12 (+); no longer U14C1.3 (+), U14D1.3 (+)
- net VCC: now also U15B1.16 (VCC)
- net at C3.1, C307.1, R303.2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: now also U3B1.27 (VCC)
- net at C332.1, C334.1, C335.2: now also U14B1.6 (-), U14B1.7; no longer U14B1.1, U14B1.2 (-)
- net at C333.1, Q331.2 (S), Q931.2 (S)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: now also U14B1.5 (+); no longer U14B1.3 (+)
- net at C331.1, Q331.1 (D), Q931.1 (D)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: now also U14C1.8; no longer U14C1.1
- net at C331.2, E305.3, R331.2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: now also U14C1.9 (-); no longer U14C1.2 (-)
- net at C321.1, Q321.1 (D), Q921.1 (D)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: now also U14D1.14; no longer U14D1.1
- net at C321.2, E306.3, R321.2: now also U14D1.13 (-); no longer U14D1.2 (-)
