File: src/cias.kicad_sch (KiCad schematic)
At the start: 78 parts, among them CN13 KEYBOARD, CN6 SERIAL_DB25M, CN7 PARALLEL_DB25F, J90 DRIVE_SWITCHER, J99 CONN_HDACT, Q501 2N3904, Q502 2N3906, Q503 2N3906, Q711 2N3904, Q99 2N3906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

Commit message: changed silkscreen thickness
Connections:
- net +12V: no longer U38E1.14 (VCC)
- net -12V: no longer U38E1.1 (VEE)
- net GND: no longer U38E1.7 (GND), U39E1.7 (GND), U42B1.1 (GND), U7B1.1 (GND), U8B1.1 (GND)
- net VCC: now also U7B1.6 (PA4), U8B1.6 (PA4); no longer U38B1.5 (IN2_B), U38C1.10 (IN1_C), U38D1.13 (IN1_D), U39E1.14 (VCC), U42B1.8 (VCC), U7B1.20 (VCC), U8B1.20 (VCC)
- net ~{TXD}: no longer U38C1.9 (IN2_C)
- net at U8A1.5 (PA3): now also U39C1.3 (OUT_A); no longer U39C1.8 (OUT_C)
- net at U8A1.6 (PA4): now also U39B1.3 (OUT_A); no longer U39B1.6 (OUT_B)
- net at U8A1.7 (PA5): now also U39D1.3 (OUT_A); no longer U39D1.11 (OUT_D)
- net at U8A1.8 (PA6): no longer U38B1.4 (IN1_B)
- net at U8A1.9 (PA7): no longer U38D1.12 (IN2_D)
- net at E532.1: now also U38C1.3; no longer U38C1.8 (OUT_C)
- net at E533.1: now also U38B1.3; no longer U38B1.6 (OUT_B)
- net at E535.1: now also U39B1.1 (IN_A); no longer U39B1.4 (IN_B)
- net at E536.1: now also U39C1.1 (IN_A); no longer U39C1.10 (IN_C)
- net at E537.1: now also U39D1.1 (IN_A); no longer U39D1.13 (IN_D)
- net at E531.1: now also U38D1.3; no longer U38D1.11 (OUT_D)
Other:
- moved on the sheet: C39, C7, C8, J90
