File: src/cias.kicad_sch (KiCad schematic)
At the start: 78 parts, among them CN13 KEYBOARD, CN6 SERIAL_DB25M, CN7 PARALLEL_DB25F, J90 DRIVE_SWITCHER, J99 CONN_HDACT, Q501 2N3904, Q502 2N3906, Q503 2N3906, Q711 2N3904, Q99 2N3906, U38B1 MC1488, U38C1 MC1488, U38D1 MC1488, U38E1 MC1488, U39A1 MC1489, U39B1 MC1489, U39C1 MC1489, U39D1 MC1489, U39E1 MC1489, U42A1 NE555, U42B1 NE555, U7A1 VIA_8520, U7B1 VIA_8520, U8A1 VIA_8520, U8B1 VIA_8520

Commit message: kicad 10
Connections:
- net +12V: now also U38E1.14 (VCC)
- net -12V: now also U38E1.1 (VEE)
- net GND: now also U38E1.7 (GND), U39E1.7 (GND), U42B1.1 (GND), U7B1.1 (GND), U8B1.1 (GND)
- net VCC: now also U38B1.5 (IN2_B), U38C1.10 (IN1_C), U38D1.13 (IN1_D), U39E1.14 (VCC), U42B1.8 (VCC), U7B1.20 (VCC), U8B1.20 (VCC); no longer U7B1.6 (PA4), U8B1.6 (PA4)
- net ~{TXD}: now also U38C1.9 (IN2_C)
- net at U8A1.5 (PA3): now also U39C1.8 (OUT_C); no longer U39C1.3 (OUT_A)
- net at U8A1.6 (PA4): now also U39B1.6 (OUT_B); no longer U39B1.3 (OUT_A)
- net at U8A1.7 (PA5): now also U39D1.11 (OUT_D); no longer U39D1.3 (OUT_A)
- net at U8A1.8 (PA6): now also U38B1.4 (IN1_B)
- net at U8A1.9 (PA7): now also U38D1.12 (IN2_D)
- net at E532.1: now also U38C1.8 (OUT_C); no longer U38C1.3
- net at E533.1: now also U38B1.6 (OUT_B); no longer U38B1.3
- net at E535.1: now also U39B1.4 (IN_B); no longer U39B1.1 (IN_A)
- net at E536.1: now also U39C1.10 (IN_C); no longer U39C1.1 (IN_A)
- net at E537.1: now also U39D1.13 (IN_D); no longer U39D1.1 (IN_A)
- net at E531.1: now also U38D1.11 (OUT_D); no longer U38D1.3
