File: src/floppy.kicad_sch (KiCad schematic)
At the start: 28 parts, among them CN11 INTERNAL_FLOPPY, CN12 FLOPPY_POWER, CN14 IDE_POWER, CN15 IDE_I/F, CN5 EXTFLOPPY_DB23F, U36A1 74LS05, U36B1 74LS05, U36C1 74LS05, U36D1 74LS05, U5B1 GARY_5719

Commit message: changed silkscreen thickness
Parts:
- renumbered CN11 to CN?, CN5 to CN?, CN15 to CN?, CN14 to CN?, CN12 to CN?, E613 to E?, E614 to E?, E615 to E?, E616 to E?, E601 to E?, E611 to E?, E612 to E?, E617 to E?, E618 to E?, E619 to E?, E620 to E?, E621 to E?, E622 to E?, E623 to E?, E624 to E?, E625 to E?, E626 to E?, E602 to E?, U36A1 to U36A?, U36B1 to U36B?, U36C1 to U36C?, U36D1 to U36D?, U5B1 to U5B?
Connections:
- net DKWE: no longer U5B?.8 (DKWE)
- net ~{DKWDB}: now also U36C?.2; no longer U36C?.6
- net ~{DKWD}: no longer U5B?.9 (~{DKWD})
- net ~{DKWEB}: now also U36D?.2; no longer U36D?.8
- net ~{KBRESET}: no longer U5B?.5 (~{KBRESET})
- net ~{MTR0}: now also U36B?.2; no longer U36B?.4
- net ~{MTR}: no longer U5B?.7 (~{MTR})
- net ~{SEL0}: no longer U5B?.16 (~{SEL})
- net at U36A?.1: no longer U5B?.47 (MTRX)
Other:
- moved on the sheet: CN?, E?, U36A?A, U36B?A, U36C?A, U36D?A
