File: src/floppy.kicad_sch (KiCad schematic)
At the start: 28 parts, among them U36A? 74LS05, U36B? 74LS05, U36C? 74LS05, U36D? 74LS05, U5B? GARY_5719

Commit message: kicad 10
Parts:
- gave numbers to parts that had none: 28
Connections:
- net DKWE: now also U5B1.8 (DKWE)
- net ~{DKWDB}: now also U36C1.6; no longer U36C1.2
- net ~{DKWD}: now also U5B1.9 (~{DKWD})
- net ~{DKWEB}: now also U36D1.8; no longer U36D1.2
- net ~{KBRESET}: now also U5B1.5 (~{KBRESET})
- net ~{MTR0}: now also U36B1.4; no longer U36B1.2
- net ~{MTR}: now also U5B1.7 (~{MTR})
- net ~{SEL0}: now also U5B1.16 (~{SEL})
- net at U36A1.1: now also U5B1.47 (MTRX)
- new net: U36D1.9, U5B1.44 (DKWEB)
- new net: U36C1.5, U5B1.45 (DKWDB)
- new net: U36B1.3, U5B1.46 (MTRON)
